File: sensor.kicad_pcb (KiCad board)
At the start: 2 copper layers, 38.7 x 42.8 mm, 18 parts, among them IC1 AP7335-WG-7, J1 Conn_01x08, U2 PMW3610

Commit message: cleanup
Parts:
- gave numbers to parts that had none: 2
Changed lines of the file:
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@@
   (footprint "" (layer "F.Cu")
     (at 81.648 92.181999)
-    (fp_text reference "" (at 0 0) (layer "F.SilkS")
+    (fp_text reference "H1" (at 0 0) (layer "F.SilkS")
         (effects (font (size 1.27 1.27) (thickness 0.15)))
     )
@@
   (footprint "" (layer "F.Cu")
     (at 81.638 129.171999)
-    (fp_text reference "" (at 0 0) (layer "F.SilkS")
+    (fp_text reference "H2" (at 0 0) (layer "F.SilkS")
         (effects (font (size 1.27 1.27) (thickness 0.15)))
     )
@@
   (gr_text "VCC" (at 96.914934 116.7) (layer "F.SilkS")
     (effects (font (face "Fira Sans") (size 1 1) (thickness 0.15)))
-    (render_cache "VCC" -0
+    (render_cache "VCC" 0
       (polygon
         (pts
@@
   (gr_text "NCS" (at 96.825541 114.16) (layer "F.SilkS")
     (effects (font (face "Fira Sans") (size 1 1) (thickness 0.15)))
-    (render_cache "NCS" -0
+    (render_cache "NCS" 0
       (polygon
         (pts
@@
   (gr_text "SCLK" (at 96.535869 109.08) (layer "F.SilkS")
     (effects (font (face "Fira Sans") (size 1 1) (thickness 0.15)))
-    (render_cache "SCLK" -0
+    (render_cache "SCLK" 0
       (polygon
         (pts
@@
   (gr_text "GND" (at 96.7 104) (layer "F.SilkS")
     (effects (font (face "Fira Sans") (size 1 1) (thickness 0.15)))
-    (render_cache "GND" -0
+    (render_cache "GND" 0
       (polygon
         (pts
@@
   (gr_text "Charybdis PMW3610 adapter\nREV 1.0" (at 73.3 98.8) (layer "F.SilkS")
     (effects (font (face "Fira Sans") (size 0.8 0.8) (thickness 0.1)) (justify left bottom))
-    (render_cache "Charybdis PMW3610 adapter\nREV 1.0" -0
+    (render_cache "Charybdis PMW3610 adapter\nREV 1.0" 0
       (polygon
         (pts
@@
   (gr_text "SDIO" (at 96.547593 111.62) (layer "F.SilkS")
     (effects (font (face "Fira Sans") (size 1 1) (thickness 0.15)))
-    (render_cache "SDIO" -0
+    (render_cache "SDIO" 0
       (polygon
         (pts
@@
   (gr_text "MO" (at 97.04829 106.54) (layer "F.SilkS")
     (effects (font (face "Fira Sans") (size 1 1) (thickness 0.15)))
-    (render_cache "MO" -0
+    (render_cache "MO" 0
       (polygon
         (pts
